File: Transistor_3X_Trigger.kicad_sch (KiCad schematic)
At the start: 8 parts, among them J1 Conn_01x01_Pin, J2 Conn_01x01_Pin, J4 Conn_01x01_Pin, J5 Conn_01x01_Pin, J6 Conn_01x01_Pin, U1 74HC14N_652

Commit message: extra commits found
Parts:
- U1: value 74HC14N_652 -> MC74HC04N_652
Other:
- note added: "must use NON-HYSTERESIS chip 74HC04N ONLY!!"
Changed lines of the file:
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@@
+		)
+	)
+	(text "must use NON-HYSTERESIS chip 74HC04N ONLY!!"
+		(exclude_from_sim no)
+		(at 162.306 136.144 0)
+		(effects
+			(font
+				(size 1.27 1.27)
+				(thickness 0.254)
+				(bold yes)
+			)
 		)
 	)
@@
 			)
 		)
-		(property "Value" "74HC14N_652"
+		(property "Value" "MC74HC04N_652"
 			(at 149.86 97.79 0)
 			(effects
